File: yacc46.kicad_pcb (KiCad board)
At the start: 2 copper layers, 281.1 x 112.1 mm, 142 parts, among them J1 USB_C_Receptacle_USB2.0, J2 OLED_I2C, J3 AVR-ISP-6, J4 GLOVE_I2C, J5 TRRS_I2C, SW1 SW_PUSH, SW10 SW_PUSH, SW11 SW_PUSH, SW12 SW_PUSH, SW13 SW_PUSH, SW14 SW_PUSH, SW15 SW_PUSH, SW16 SW_PUSH, SW17 SW_PUSH, SW18 SW_PUSH, SW19 Rotary_Encoder_Switch, SW2 SW_PUSH, SW20 SW_PUSH, SW21 SW_PUSH, SW22 SW_PUSH, SW23 SW_PUSH, SW24 SW_PUSH, SW25 SW_PUSH, SW26 SW_PUSH, SW27 SW_PUSH, SW28 SW_PUSH, SW29 SW_PUSH, SW3 SW_PUSH, SW30 SW_PUSH, SW31 SW_PUSH, SW32 SW_PUSH, SW33 SW_PUSH, SW34 SW_PUSH, SW35 SW_PUSH, SW36 Rotary_Encoder_Switch, SW37 SW_PUSH, SW38 SW_PUSH, SW39 SW_PUSH, SW4 SW_PUSH, SW40 SW_PUSH, SW41 SW_PUSH, SW42 SW_PUSH, SW43 SW_PUSH, SW44 SW_PUSH, SW45 SW_PUSH, SW46 SW_PUSH, SW47 SW_Push, SW5 SW_PUSH, SW6 SW_PUSH, SW7 SW_PUSH, SW8 SW_PUSH, SW9 SW_PUSH, U1 ATmega32U4-AU, Y1 16MHz

Commit message: 微修正
Parts:
- renumbered REF** to HOLE13, REF** to HOLE14
Routing:
- net GND: track 926.1 -> 938.2 mm
- net Net-(J1-PadB5): track 18.3 -> 18.9 mm, vias 1 -> 3

Commit message: 基板外形を変更
Parts:
- moved HOLE3 5.50 mm to (42.6, 94.9)
- moved HOLE10 5.50 mm to (286.9, 94.9)
- moved D41 5.49 mm to (285.7, 85.2)
Routing:
- net Net-(LED2-Pad3): track 96.3 -> 88.4 mm
- net COL1: track 363.9 -> 367.8 mm, vias 8 -> 7
- net ROWR2: track 318.4 -> 321.6 mm
- net ROWL2: track 184.7 -> 182.0 mm, vias 10 -> 8
- net Net-(D41-Pad2): track 5.23 -> 3.60 mm
- net Net-(LED3-Pad3): track 96.1 -> 97.4 mm, vias 3 -> 4
- net COL0: track 367.0 -> 366.3 mm, vias 8 -> 6
- net VBUS: track 857.6 -> 858.2 mm
Other:
- outline, holes or cut-outs redrawn

Commit message: USBコネクタをCX70M-24P1に変更
Parts:
- J1: value USB_C_Receptacle_USB2.0 -> CX70M-24P1; footprint 1m38_kbd:USB_C_Receptacle_GCT_USB4085 -> digikey-footprints:USB-C_Female_CX70M-24P1
- moved J1 4.25 mm to (31.5, 50.8)
- moved R1 1.87 mm to (39.4, 49.9)
- moved R2 1.87 mm to (39.4, 52.4), turned to 0 degrees
Connections:
- net /DUN renamed UDN
- net /DUP renamed UDP
- net Net-(F1-Pad2) renamed UVBUS
- net Net-(J1-PadA5) renamed /CC1
- J1 pad B5: Net-(J1-PadB5) -> /CC2
- R2 pad 1: GND -> /CC2
- R2 pad 2: Net-(J1-PadB5) -> GND
Routing:
- net UVBUS: track 28.9 -> 59.4 mm, vias 0 -> 2
- net Net-(J1-PadB5): track 18.9 -> 0.00 mm, vias 3 -> 0
- net /CC2: track 0.00 -> 7.76 mm
- net UDP: track 233.6 -> 239.9 mm, vias 3 -> 4
- net UDN: track 232.8 -> 236.6 mm, vias 3 -> 4
- net GND: track 938.2 -> 941.3 mm, vias 11 -> 13
- net /CC1: track 7.01 -> 6.77 mm, vias 0 -> 1
Other:
- outline, holes or cut-outs redrawn
- net class Receptacle added: clearance 0.17, trace_width 0.23, via_dia 0.8, via_drill 0.4
- rule trace_min: 0.2032 -> 0.1524

Commit message: おおよそPCBの最終調整完了
Parts:
- R1, R2, R3, R4, R5, R6: footprint Resistor_SMD:R_0603_1608Metric_Pad1.05x0.95mm_HandSolder -> Resistor_SMD:R_0805_2012Metric_Pad1.15x1.40mm_HandSolder
- SW47: footprint foostan-kbd:ResetSW_1side -> 1m38_kbd:ResetSW_SKRPABE010; moved to B.Cu
- moved R6 3.82 mm to (152.9, 133.1), turned to 0 degrees
- moved HOLE13 2.06 mm to (152.0, 60.1)
- moved HOLE14 2.06 mm to (177.5, 60.1)
- moved SW47 2.05 mm to (186.0, 134.2), turned to 0 degrees
- moved R5 1.73 mm to (186.0, 130.1)
Routing:
- net COL3: track 335.4 -> 341.0 mm, vias 5 -> 7
- net GND: track 941.3 -> 946.2 mm, vias 13 -> 16
- net RESET: track 174.0 -> 170.5 mm
- net SDA: track 271.4 -> 268.4 mm
- net SCL: track 266.5 -> 263.7 mm
- net ROWL2: track 182.0 -> 183.8 mm
- net COL6: track 159.7 -> 161.5 mm, vias 5 -> 6
- net HWB: track 12.8 -> 11.2 mm
- net ROWL3: track 75.9 -> 77.4 mm
- net VBUS: track 858.2 -> 857.1 mm
- net COL0: track 366.3 -> 367.2 mm
- net COL1: track 367.8 -> 368.7 mm, vias 7 -> 8
- net COL2: track 341.4 -> 342.3 mm, vias 7 -> 9
- net Net-(LED7-Pad3): track 107.6 -> 108.4 mm
- net MISO: track 300.4 -> 299.7 mm
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Other:
- net class Power added: clearance 0.2, trace_width 0.5, via_dia 0.8, via_drill 0.4
- board text added: "yacc46 v0.1 PCB designed by 1.038"
- board text removed: "yacc46 v0.1 designed by 1.038"
