File: yacc46_plate.kicad_pcb (KiCad board)
At the start: 2 copper layers, 281.1 x 112.1 mm, 126 parts, among them J1 USB_C_Receptacle_USB2.0, J2 OLED_I2C, J3 AVR-ISP-6, J4 GLOVE_I2C, J5 TRRS_I2C, SW1 SW_PUSH, SW10 SW_PUSH, SW11 SW_PUSH, SW12 SW_PUSH, SW13 SW_PUSH, SW14 SW_PUSH, SW15 SW_PUSH, SW16 SW_PUSH, SW17 SW_PUSH, SW18 SW_PUSH, SW19 Rotary_Encoder_Switch, SW2 SW_PUSH, SW20 SW_PUSH, SW21 SW_PUSH, SW22 SW_PUSH, SW23 SW_PUSH, SW24 SW_PUSH, SW25 SW_PUSH, SW26 SW_PUSH, SW27 SW_PUSH, SW28 SW_PUSH, SW29 SW_PUSH, SW3 SW_PUSH, SW30 SW_PUSH, SW31 SW_PUSH, SW32 SW_PUSH, SW33 SW_PUSH, SW34 SW_PUSH, SW35 SW_PUSH, SW36 Rotary_Encoder_Switch, SW37 SW_PUSH, SW38 SW_PUSH, SW39 SW_PUSH, SW4 SW_PUSH, SW40 SW_PUSH, SW41 SW_PUSH, SW42 SW_PUSH, SW43 SW_PUSH, SW44 SW_PUSH, SW45 SW_PUSH, SW46 SW_PUSH, SW5 SW_PUSH, SW6 SW_PUSH, SW7 SW_PUSH, SW8 SW_PUSH, SW9 SW_PUSH, U1 ATmega32U4-AU, Y1 16MHz

Commit message: プレートデータを作成
Parts:
- added HOLE1: Val**, foostan-kbd:M2_HOLE_v2, F.Cu at (132.0, 133.1)
- added HOLE10: Val**, foostan-kbd:M2_HOLE_v2, F.Cu at (286.9, 94.9)
- added HOLE11: Val**, foostan-kbd:M2_HOLE_v2, F.Cu at (244.9, 100.6)
- added HOLE12: Val**, foostan-kbd:M2_HOLE_v2, F.Cu at (197.6, 133.1)
- added HOLE13: MountingHole_2.2mm_M2, MountingHole:MountingHole_2.2mm_M2, F.Cu at (152.0, 60.1)
- added HOLE13: Val**, foostan-kbd:M2_HOLE_v2, F.Cu at (164.8, 88.2)
- added HOLE14: MountingHole_2.2mm_M2, MountingHole:MountingHole_2.2mm_M2, F.Cu at (177.5, 60.1)
- added HOLE2: Val**, foostan-kbd:M2_HOLE_v2, F.Cu at (84.6, 100.6)
- added HOLE3: Val**, foostan-kbd:M2_HOLE_v2, F.Cu at (42.6, 94.9)
- added HOLE4: Val**, foostan-kbd:M2_HOLE_v2, F.Cu at (39.7, 43.7)
- added HOLE5: Val**, foostan-kbd:M2_HOLE_v2, F.Cu at (86.3, 32.1)
- added HOLE6: Val**, foostan-kbd:M2_HOLE_v2, F.Cu at (142.0, 31.8)
- added HOLE7: Val**, foostan-kbd:M2_HOLE_v2, F.Cu at (187.6, 31.8)
- added HOLE8: Val**, foostan-kbd:M2_HOLE_v2, F.Cu at (243.2, 32.1)
- added HOLE9: Val**, foostan-kbd:M2_HOLE_v2, F.Cu at (289.8, 43.7)
- J1: value USB_C_Receptacle_USB2.0 -> CX70M-24P1; footprint 1m38_kbd:USB_C_Receptacle_GCT_USB4085 -> digikey-footprints:USB-C_Female_CX70M-24P1
- R1, R2, R3, R4, R5, R6: footprint Resistor_SMD:R_0603_1608Metric_Pad1.05x0.95mm_HandSolder -> Resistor_SMD:R_0805_2012Metric_Pad1.15x1.40mm_HandSolder
- SW1, SW10, SW11, SW12, SW13, SW14, SW15, SW16, SW17, SW18, SW19, SW2, SW20, SW21, SW22, SW23, SW24, SW25, SW26, SW27, SW28, SW29, SW3, SW30, SW31, SW32, SW33, SW34, SW35, SW36, SW37, SW38, SW39, SW4, SW40, SW41, SW42, SW43, SW44, SW45, SW46, SW5, SW6, SW7, SW8, SW9: footprint foostan-kbd:SW_Hole -> 1m38_kbd:CherryMX_SwitchHole_RoundCorner
- moved J1 4.25 mm to (31.5, 50.8)
- moved R6 3.82 mm to (152.9, 133.1), turned to 0 degrees
- moved R1 1.87 mm to (39.4, 49.9)
- moved R2 1.87 mm to (39.4, 52.4), turned to 0 degrees
- moved R5 1.73 mm to (186.0, 130.1)
Connections:
- net /DUN renamed UDN
- net /DUP renamed UDP
- net Net-(F1-Pad2) renamed UVBUS
- net Net-(J1-PadA5) renamed /CC1
- J1 pad B5: Net-(J1-PadB5) -> /CC2
- R2 pad 1: GND -> /CC2
- R2 pad 2: Net-(J1-PadB5) -> GND
Other:
- outline, holes or cut-outs redrawn
- net class Power added: clearance 0.2, trace_width 0.5, via_dia 0.8, via_drill 0.4
- net class Receptacle added: clearance 0.17, trace_width 0.23, via_dia 0.8, via_drill 0.4
- rule trace_min: 0.2032 -> 0.1524
- board text added: "yacc46 v0.1 PCB designed by 1.038"
