File: yacc46/yacc46.sch (KiCad schematic (older format))
At the start: 139 parts, among them J1 USB_C_Receptacle_USB2.0, J2 OLED_I2C, J3 AVR-ISP-6, J4 GLOVE_I2C, SW1 SW_PUSH, SW10 SW_PUSH, SW11 SW_PUSH, SW12 SW_PUSH, SW13 SW_PUSH, SW14 SW_PUSH, SW15 SW_PUSH, SW16 SW_PUSH, SW17 SW_PUSH, SW18 SW_PUSH, SW19 Rotary_Encoder_Switch, SW2 SW_PUSH, SW20 SW_PUSH, SW21 SW_PUSH, SW22 SW_PUSH, SW23 SW_PUSH, SW24 SW_PUSH, SW25 SW_PUSH, SW26 SW_PUSH, SW27 SW_PUSH, SW28 SW_PUSH, SW29 SW_PUSH, SW3 SW_PUSH, SW30 SW_PUSH, SW31 SW_PUSH, SW32 SW_PUSH, SW33 SW_PUSH, SW34 SW_PUSH, SW35 SW_PUSH, SW36 Rotary_Encoder_Switch, SW37 SW_PUSH, SW38 SW_PUSH, SW39 SW_PUSH, SW4 SW_PUSH, SW40 SW_PUSH, SW41 SW_PUSH, SW42 SW_PUSH, SW43 SW_PUSH, SW44 SW_PUSH, SW45 SW_PUSH, SW46 SW_PUSH, SW47 SW_Push, SW5 SW_PUSH, SW6 SW_PUSH, SW7 SW_PUSH, SW8 SW_PUSH, SW9 SW_PUSH, U1 ATmega32U4-AU, Y1 16MHz

Commit message: yacc46 回路図: LED13,14を忘れていたので追加
Parts:
- added LED13, LED14: WS2812B, foostan_kbd:LED_WS2812B-PLCC4, symbol LED:WS2812B
Connections:
- net GND: now also LED13.3 (VSS), LED14.3 (VSS)
- net VCC: now also LED13.1 (VDD), LED14.1 (VDD)
- net at LED12.2 (DOUT): now also LED13.4 (DIN)
- new net: LED13.2 (DOUT), LED14.4 (DIN)
Other:
- moved on the sheet: LED10, LED11, LED12, LED8, LED9
Changed lines of the file:
@@
 L power:VCC #PWR019
 U 1 1 5FB87C1E
-P 4850 8600
-F 0 "#PWR019" H 4850 8450 50  0001 C CNN
-F 1 "VCC" H 4865 8773 50  0000 C CNN
-F 2 "" H 4850 8600 50  0001 C CNN
-F 3 "" H 4850 8600 50  0001 C CNN
-	1    4850 8600
+P 4700 8650
+F 0 "#PWR019" H 4700 8500 50  0001 C CNN
+F 1 "VCC" H 4715 8823 50  0000 C CNN
+F 2 "" H 4700 8650 50  0001 C CNN
+F 3 "" H 4700 8650 50  0001 C CNN
+	1    4700 8650
 	1    0    0    -1
 $EndComp
@@
 L power:GND #PWR021
 U 1 1 5FC0B3A4
-P 4850 9300
-F 0 "#PWR021" H 4850 9050 50  0001 C CNN
-F 1 "GND" H 4855 9127 50  0000 C CNN
-F 2 "" H 4850 9300 50  0001 C CNN
-F 3 "" H 4850 9300 50  0001 C CNN
-	1    4850 9300
+P 4700 9250
+F 0 "#PWR021" H 4700 9000 50  0001 C CNN
+F 1 "GND" H 4705 9077 50  0000 C CNN
+F 2 "" H 4700 9250 50  0001 C CNN
+F 3 "" H 4700 9250 50  0001 C CNN
+	1    4700 9250
 	1    0    0    -1
 $EndComp
@@
 L LED:WS2812B LED8
 U 1 1 606C75EF
-P 10650 8950
-F 0 "LED8" H 10900 8800 50  0000 L CNN
-F 1 "WS2812B" H 10900 8700 50  0000 L CNN
-F 2 "foostan_kbd:LED_WS2812B-PLCC4" H 10700 8650 50  0001 L TNN
-F 3 "https://cdn-shop.adafruit.com/datasheets/WS2812B.pdf" H 10750 8575 50  0001 L TNN
-	1    10650 8950
+P 5050 10050
+F 0 "LED8" H 5300 9900 50  0000 L CNN
+F 1 "WS2812B" H 5300 9800 50  0000 L CNN
+F 2 "foostan_kbd:LED_WS2812B-PLCC4" H 5100 9750 50  0001 L TNN
+F 3 "https://cdn-shop.adafruit.com/datasheets/WS2812B.pdf" H 5150 9675 50  0001 L TNN
+	1    5050 10050
 	1    0    0    -1
 $EndComp
@@
 L LED:WS2812B LED9
 U 1 1 606C7EB9
-P 11450 8950
-F 0 "LED9" H 11700 8800 50  0000 L CNN
-F 1 "WS2812B" H 11700 8700 50  0000 L CNN
-F 2 "foostan_kbd:LED_WS2812B-PLCC4" H 11500 8650 50  0001 L TNN
-F 3 "https://cdn-shop.adafruit.com/datasheets/WS2812B.pdf" H 11550 8575 50  0001 L TNN
-	1    11450 8950
+P 5850 10050
+F 0 "LED9" H 6100 9900 50  0000 L CNN
+F 1 "WS2812B" H 6100 9800 50  0000 L CNN
+F 2 "foostan_kbd:LED_WS2812B-PLCC4" H 5900 9750 50  0001 L TNN
+F 3 "https://cdn-shop.adafruit.com/datasheets/WS2812B.pdf" H 5950 9675 50  0001 L TNN
+	1    5850 10050
 	1    0    0    -1
 $EndComp
@@
 L LED:WS2812B LED10
 U 1 1 606C864B
-P 12250 8950
-F 0 "LED10" H 12500 8800 50  0000 L CNN
-F 1 "WS2812B" H 12500 8700 50  0000 L CNN
-F 2 "foostan_kbd:LED_WS2812B-PLCC4" H 12300 8650 50  0001 L TNN
-F 3 "https://cdn-shop.adafruit.com/datasheets/WS2812B.pdf" H 12350 8575 50  0001 L TNN
-	1    12250 8950
+P 6650 10050
+F 0 "LED10" H 6900 9900 50  0000 L CNN
+F 1 "WS2812B" H 6900 9800 50  0000 L CNN
+F 2 "foostan_kbd:LED_WS2812B-PLCC4" H 6700 9750 50  0001 L TNN
+F 3 "https://cdn-shop.adafruit.com/datasheets/WS2812B.pdf" H 6750 9675 50  0001 L TNN
+	1    6650 10050
 	1    0    0    -1
 $EndComp
@@
 L LED:WS2812B LED11
 U 1 1 606C8C99
-P 13050 8950
-F 0 "LED11" H 13300 8800 50  0000 L CNN
-F 1 "WS2812B" H 13300 8700 50  0000 L CNN
-F 2 "foostan_kbd:LED_WS2812B-PLCC4" H 13100 8650 50  0001 L TNN
-F 3 "https://cdn-shop.adafruit.com/datasheets/WS2812B.pdf" H 13150 8575 50  0001 L TNN
-	1    13050 8950
+P 7450 10050
+F 0 "LED11" H 7700 9900 50  0000 L CNN
+F 1 "WS2812B" H 7700 9800 50  0000 L CNN
+F 2 "foostan_kbd:LED_WS2812B-PLCC4" H 7500 9750 50  0001 L TNN
+F 3 "https://cdn-shop.adafruit.com/datasheets/WS2812B.pdf" H 7550 9675 50  0001 L TNN
+	1    7450 10050
 	1    0    0    -1
 $EndComp
@@
 L LED:WS2812B LED12
 U 1 1 606C9449
-P 13850 8950
-F 0 "LED12" H 14100 8800 50  0000 L CNN
-F 1 "WS2812B" H 14100 8700 50  0000 L CNN
-F 2 "foostan_kbd:LED_WS2812B-PLCC4" H 13900 8650 50  0001 L TNN
-F 3 "https://cdn-shop.adafruit.com/datasheets/WS2812B.pdf" H 13950 8575 50  0001 L TNN
-	1    13850 8950
+P 8250 10050
+F 0 "LED12" H 8500 9900 50  0000 L CNN
+F 1 "WS2812B" H 8500 9800 50  0000 L CNN
+F 2 "foostan_kbd:LED_WS2812B-PLCC4" H 8300 9750 50  0001 L TNN
+F 3 "https://cdn-shop.adafruit.com/datasheets/WS2812B.pdf" H 8350 9675 50  0001 L TNN
+	1    8250 10050
 	1    0    0    -1
 $EndComp
@@
 	9350 8950 9550 8950
 Wire Wire Line
-	10150 8950 10350 8950
-Wire Wire Line
-	10950 8950 11150 8950
-Wire Wire Line
-	11750 8950 11950 8950
-Wire Wire Line
-	12550 8950 12750 8950
-Wire Wire Line
-	13350 8950 13550 8950
-NoConn ~ 14150 8950
+	4550 10050 4750 10050
+Wire Wire Line
+	5350 10050 5550 10050
+Wire Wire Line
+	6150 10050 6350 10050
+Wire Wire Line
+	6950 10050 7150 10050
+Wire Wire Line
+	7750 10050 7950 10050
 Wire Wire Line
 	5050 8650 5850 8650
@@
 Wire Wire Line
 	9050 8650 9850 8650
-Connection ~ 9850 8650
-Wire Wire Line
-	9850 8650 10650 8650
-Connection ~ 10650 8650
-Wire Wire Line
-	10650 8650 11450 8650
-Connection ~ 11450 8650
-Wire Wire Line
-	11450 8650 12250 8650
-Connection ~ 12250 8650
-Wire Wire Line
-	12250 8650 13050 8650
-Connection ~ 13050 8650
-Wire Wire Line
-	13050 8650 13850 8650
+Wire Wire Line
+	5050 9750 5850 9750
+Connection ~ 5850 9750
+Wire Wire Line
+	5850 9750 6650 9750
+Connection ~ 6650 9750
+Wire Wire Line
+	6650 9750 7450 9750
+Connection ~ 7450 9750
+Wire Wire Line
+	7450 9750 8250 9750
 Wire Wire Line
 	5050 9250 5850 9250
@@
 Wire Wire Line
 	9050 9250 9850 9250
-Connection ~ 9850 9250
-Wire Wire Line
-	9850 9250 10650 9250
-Connection ~ 10650 9250
-Wire Wire Line
-	10650 9250 11450 9250
-Connection ~ 11450 9250
-Wire Wire Line
-	11450 9250 12250 9250
-Connection ~ 12250 9250
-Wire Wire Line
-	12250 9250 13050 9250
-Connection ~ 13050 9250
-Wire Wire Line
-	13050 9250 13850 9250
-Wire Wire Line
-	4850 9300 4850 9250
-Wire Wire Line
-	4850 9250 5050 9250
+Wire Wire Line
+	5050 10350 5850 10350
+Connection ~ 5850 10350
+Wire Wire Line
+	5850 10350 6650 10350
+Connection ~ 6650 10350
+Wire Wire Line
+	6650 10350 7450 10350
+Connection ~ 7450 10350
+Wire Wire Line
+	7450 10350 8250 10350
 Connection ~ 5050 9250
-Wire Wire Line
-	4850 8600 4850 8650
-Wire Wire Line
-	4850 8650 5050 8650
 Connection ~ 5050 8650
 $Comp
@@
 	1    0    0    -1
 $EndComp
+$Comp
+L LED:WS2812B LED13
+U 1 1 60753107
+P 9050 10050
+F 0 "LED13" H 9300 9900 50  0000 L CNN
+F 1 "WS2812B" H 9300 9800 50  0000 L CNN
+F 2 "foostan_kbd:LED_WS2812B-PLCC4" H 9100 9750 50  0001 L TNN
+F 3 "https://cdn-shop.adafruit.com/datasheets/WS2812B.pdf" H 9150 9675 50  0001 L TNN
+	1    9050 10050
+	1    0    0    -1
+$EndComp
+$Comp
+L LED:WS2812B LED14
+U 1 1 60753913
+P 9850 10050
+F 0 "LED14" H 10100 9900 50  0000 L CNN
+F 1 "WS2812B" H 10100 9800 50  0000 L CNN
+F 2 "foostan_kbd:LED_WS2812B-PLCC4" H 9900 9750 50  0001 L TNN
+F 3 "https://cdn-shop.adafruit.com/datasheets/WS2812B.pdf" H 9950 9675 50  0001 L TNN
+	1    9850 10050
+	1    0    0    -1
+$EndComp
+NoConn ~ 10150 10050
+Wire Wire Line
+	8550 10050 8750 10050
+Wire Wire Line
+	9350 10050 9550 10050
+Wire Wire Line
+	8250 9750 9050 9750
+Connection ~ 8250 9750
+Connection ~ 9050 9750
+Wire Wire Line
+	9050 9750 9850 9750
+Wire Wire Line
+	8250 10350 9050 10350
+Connection ~ 8250 10350
+Connection ~ 9050 10350
+Wire Wire Line
+	9050 10350 9850 10350
+Wire Wire Line
+	10150 8950 10550 8950
+Wire Wire Line
+	10550 8950 10550 9500
+Wire Wire Line
+	10550 9500 4550 9500
+$Comp
+L power:VCC #PWR05
+U 1 1 607E3C62
+P 4700 9750
+F 0 "#PWR05" H 4700 9600 50  0001 C CNN
+F 1 "VCC" H 4715 9923 50  0000 C CNN
+F 2 "" H 4700 9750 50  0001 C CNN
+F 3 "" H 4700 9750 50  0001 C CNN
+	1    4700 9750
+	1    0    0    -1
+$EndComp
+Wire Wire Line
+	4700 9750 5050 9750
+Connection ~ 5050 9750
+$Comp
+L power:GND #PWR07
+U 1 1 607F8EE4
+P 4700 10350
+F 0 "#PWR07" H 4700 10100 50  0001 C CNN
+F 1 "GND" H 4705 10177 50  0000 C CNN
+F 2 "" H 4700 10350 50  0001 C CNN
+F 3 "" H 4700 10350 50  0001 C CNN
+	1    4700 10350
+	1    0    0    -1
+$EndComp
+Wire Wire Line
+	4700 10350 5050 10350
+Connection ~ 5050 10350
+Wire Wire Line
+	4700 9250 5050 9250
+Wire Wire Line
+	4700 8650 5050 8650
+Wire Wire Line
+	4550 9500 4550 10050
 $EndSCHEMATC

Commit message: yacc46 回路図: Switchジョイコンのジョイスティックを追加 (ピン配置は仮)
Parts:
- added J3: joystick_switch_joycon, symbol 1m38_kbd:joystick_switch_joycon
- renumbered J3 to J4, J4 to J5
Connections:
- net ENCL1: now also U1.36 (PF7); no longer U1.38 (PF5)
- net ENCL2: now also U1.37 (PF6); no longer U1.39 (PF4)
- net ENCR1: now also U1.39 (PF4); no longer U1.41 (PF0)
- net ENCR2: now also U1.38 (PF5); no longer U1.40 (PF1)
- net GND: now also J3.2 (GND)
- net ROWL0: now also U1.12 (PB7); no longer U1.37 (PF6)
- net ROWL1: now also U1.20 (PD2); no longer U1.36 (PF7)
- net VCC: now also J3.5 (Vcc)
- net JOYSTBT: now reaches U1.1 (PE6)
- net JOYSTBT: now also J3.3 (BTN)
- new net JOYSTX: J3.1 (X), U1.41 (PF0)
- new net JOYSTY: J3.4 (Y), U1.40 (PF1)
- no-connect marks 6 -> 3
Changed lines of the file:
@@
 Text GLabel 6350 1800 2    50   Input ~ 0
 COL6
-Text GLabel 6350 3700 2    50   Input ~ 0
+Text GLabel 6350 3900 2    50   Input ~ 0
 ENCR1
-Text GLabel 6350 3800 2    50   Input ~ 0
+Text GLabel 6350 4000 2    50   Input ~ 0
 ENCR2
-Text GLabel 6350 4000 2    50   Input ~ 0
+Text GLabel 6350 4200 2    50   Input ~ 0
 ENCL1
-Text GLabel 6350 3900 2    50   Input ~ 0
+Text GLabel 6350 4100 2    50   Input ~ 0
 ENCL2
 Text GLabel 6350 1900 2    50   Input ~ 0
@@
 $EndComp
 $Comp
-L Connector:AVR-ISP-6 J3
+L Connector:AVR-ISP-6 J4
 U 1 1 5F784B6C
 P 1500 9000
-F 0 "J3" H 1171 9096 50  0000 R CNN
+F 0 "J4" H 1171 9096 50  0000 R CNN
 F 1 "AVR-ISP-6" H 1171 9005 50  0000 R CNN
 F 2 "1m38_kbd:ICSP-Header-ZigZag-Single" V 1250 9050 50  0001 C CNN
@@
 Wire Wire Line
 	6400 1450 6850 1450
-NoConn ~ 6350 3500
 Wire Wire Line
 	3850 4450 3900 4450
@@
 	3000 8900 3000 9000
 $Comp
-L Connector_Generic:Conn_01x04 J4
+L Connector_Generic:Conn_01x04 J5
 U 1 1 5F59F101
 P 2800 8700
-F 0 "J4" V 3000 8400 50  0000 R CNN
+F 0 "J5" V 3000 8400 50  0000 R CNN
 F 1 "GLOVE_I2C" V 2900 8400 50  0000 R CNN
 F 2 "1m38_kbd:Grove_I2C" H 2800 8700 50  0001 C CNN
@@
 Text GLabel 6450 1500 2    50   Input ~ 0
 ROWR1
-Text GLabel 6350 4200 2    50   Input ~ 0
+Text GLabel 6600 2700 2    50   Input ~ 0
 ROWL1
 Text GLabel 6350 2300 2    50   Input ~ 0
@@
 Wire Wire Line
 	8200 7500 9000 7500
-Text GLabel 6350 4100 2    50   Input ~ 0
+Text GLabel 6600 2000 2    50   Input ~ 0
 ROWL0
 Text GLabel 6850 1650 2    50   Input ~ 0
@@
 	6450 1600 6400 1600
 Connection ~ 6400 1600
-NoConn ~ 6350 2000
-NoConn ~ 6350 2700
 Connection ~ 5750 4600
 Wire Wire Line
@@
 Wire Wire Line
 	4550 9500 4550 10050
+$Comp
+L 1m38_kbd:joystick_switch_joycon J3
+U 1 1 609C0DD2
+P 7050 7800
+F 0 "J3" H 7478 7846 50  0000 L CNN
+F 1 "joystick_switch_joycon" H 7478 7755 50  0000 L CNN
+F 2 "" H 6850 7750 50  0001 C CNN
+F 3 "" H 6850 7750 50  0001 C CNN
+	1    7050 7800
+	1    0    0    -1
+$EndComp
+$Comp
+L power:GND #PWR0107
+U 1 1 609C2EA8
+P 6100 7950
+F 0 "#PWR0107" H 6100 7700 50  0001 C CNN
+F 1 "GND" H 6105 7777 50  0000 C CNN
+F 2 "" H 6100 7950 50  0001 C CNN
+F 3 "" H 6100 7950 50  0001 C CNN
+	1    6100 7950
+	1    0    0    -1
+$EndComp
+$Comp
+L power:VCC #PWR0108
+U 1 1 609C381E
+P 6100 7500
+F 0 "#PWR0108" H 6100 7350 50  0001 C CNN
+F 1 "VCC" H 6115 7673 50  0000 C CNN
+F 2 "" H 6100 7500 50  0001 C CNN
+F 3 "" H 6100 7500 50  0001 C CNN
+	1    6100 7500
+	1    0    0    -1
+$EndComp
+Wire Wire Line
+	6100 7500 6500 7500
+Wire Wire Line
+	6100 7950 6500 7950
+Text GLabel 6350 3700 2    50   Input ~ 0
+JOYSTX
+Text GLabel 6500 8100 0    50   Input ~ 0
+JOYSTX
+Text GLabel 6350 3800 2    50   Input ~ 0
+JOYSTY
+Text GLabel 6500 7650 0    50   Input ~ 0
+JOYSTY
+Wire Wire Line
+	6350 2000 6600 2000
+Wire Wire Line
+	6350 2700 6600 2700
+Text GLabel 6600 3500 2    50   Input ~ 0
+JOYSTBT
+Wire Wire Line
+	6350 3500 6600 3500
+Text GLabel 6500 7800 0    50   Input ~ 0
+JOYSTBT
 $EndSCHEMATC

Commit message: FPCコネクタのフットプリントを作成
Parts:
- J3: footprint (none) -> 1m38_kbd:Molex_FPC_CON_0.5mm_5pin_5051100592
Changed lines of the file:
@@
 F 0 "J3" H 7478 7846 50  0000 L CNN
 F 1 "joystick_switch_joycon" H 7478 7755 50  0000 L CNN
-F 2 "" H 6850 7750 50  0001 C CNN
+F 2 "1m38_kbd:Molex_FPC_CON_0.5mm_5pin_5051100592" H 6850 7750 50  0001 C CNN
 F 3 "" H 6850 7750 50  0001 C CNN
 	1    7050 7800

Commit message: ESDダイオードのフットプリントを変更
Parts:
- D47: footprint Package_TO_SOT_SMD:SOT-143 -> 1m38_kbd:PRTR5V0U2X_SOT143B
Changed lines of the file:
@@
 F 0 "D47" V 3296 3406 50  0000 R CNN
 F 1 "PRTR5V0U2X" V 3205 3406 50  0000 R CNN
-F 2 "Package_TO_SOT_SMD:SOT-143" H 3310 3950 50  0001 C CNN
+F 2 "1m38_kbd:PRTR5V0U2X_SOT143B" H 3310 3950 50  0001 C CNN
 F 3 "https://assets.nexperia.com/documents/data-sheet/PRTR5V0U2X.pdf" H 3310 3950 50  0001 C CNN
 	1    3250 3950
