File: yacc46/yacc46.sch (KiCad schematic (older format))
At the start: 142 parts, among them J1 USB_C_Receptacle_USB2.0, J2 OLED_I2C, J3 joystick_switch_joycon, J4 AVR-ISP-6, J5 GLOVE_I2C, SW1 SW_PUSH, SW10 SW_PUSH, SW11 SW_PUSH, SW12 SW_PUSH, SW13 SW_PUSH, SW14 SW_PUSH, SW15 SW_PUSH, SW16 SW_PUSH, SW17 SW_PUSH, SW18 SW_PUSH, SW19 Rotary_Encoder_Switch, SW2 SW_PUSH, SW20 SW_PUSH, SW21 SW_PUSH, SW22 SW_PUSH, SW23 SW_PUSH, SW24 SW_PUSH, SW25 SW_PUSH, SW26 SW_PUSH, SW27 SW_PUSH, SW28 SW_PUSH, SW29 SW_PUSH, SW3 SW_PUSH, SW30 SW_PUSH, SW31 SW_PUSH, SW32 SW_PUSH, SW33 SW_PUSH, SW34 SW_PUSH, SW35 SW_PUSH, SW36 Rotary_Encoder_Switch, SW37 SW_PUSH, SW38 SW_PUSH, SW39 SW_PUSH, SW4 SW_PUSH, SW40 SW_PUSH, SW41 SW_PUSH, SW42 SW_PUSH, SW43 SW_PUSH, SW44 SW_PUSH, SW45 SW_PUSH, SW46 SW_PUSH, SW47 SW_Push, SW5 SW_PUSH, SW6 SW_PUSH, SW7 SW_PUSH, SW8 SW_PUSH, SW9 SW_PUSH, U1 ATmega32U4-AU, Y1 16MHz

Commit message: 配線完了
Connections:
- net COL0: now also U1.22 (PD5); no longer U1.21 (PD3)
- net COL1: now also U1.36 (PF7); no longer U1.22 (PD5)
- net COL2: now also U1.37 (PF6); no longer U1.25 (PD4)
- net COL3: now also J4.3 (SCK), U1.9 (PB1); no longer U1.26 (PD6)
- net COL4: now also J4.4 (MOSI), U1.10 (PB2); no longer U1.27 (PD7)
- net COL5: now also J4.1 (MISO), U1.11 (PB3); no longer U1.28 (PB4)
- net COL6: now also U1.12 (PB7); no longer U1.29 (PB5)
- net ENCL1: now also U1.29 (PB5); no longer U1.36 (PF7)
- net ENCL2: now also U1.28 (PB4); no longer U1.37 (PF6)
- net ENCR1: now also U1.41 (PF0); no longer U1.39 (PF4)
- net ENCR2: now also U1.40 (PF1); no longer U1.38 (PF5)
- net JOYSTBT: now also U1.27 (PD7); no longer U1.1 (PE6)
- net JOYSTX: now also U1.26 (PD6); no longer U1.41 (PF0)
- net JOYSTY: now also U1.25 (PD4); no longer U1.40 (PF1)
- net LED: now also U1.20 (PD2); no longer U1.30 (PB6)
- net ROWL0: now also U1.32 (PC7); no longer U1.12 (PB7)
- net ROWL1: now also U1.31 (PC6); no longer U1.20 (PD2)
- net ROWL2: now also U1.30 (PB6); no longer U1.32 (PC7)
- net ROWL3: now also U1.21 (PD3); no longer U1.31 (PC6)
- net ROWR2: now also U1.1 (PE6); no longer J4.3 (SCK), U1.9 (PB1)
- net MISO renamed ROWR0
- net ROWR0: now also U1.38 (PF5); no longer J4.1 (MISO), U1.11 (PB3)
- net MOSI renamed ROWR1
- net ROWR1: now also U1.39 (PF4); no longer J4.4 (MOSI), U1.10 (PB2)
Changed lines of the file:
@@
 Wire Wire Line
 	6400 1600 6400 1650
-Text GLabel 6350 2800 2    50   Input ~ 0
+Text GLabel 6350 3000 2    50   Input ~ 0
 COL0
-Text GLabel 6350 3000 2    50   Input ~ 0
+Text GLabel 6350 4200 2    50   Input ~ 0
 COL1
-Text GLabel 6350 2900 2    50   Input ~ 0
+Text GLabel 6350 4100 2    50   Input ~ 0
 COL2
-Text GLabel 6350 3100 2    50   Input ~ 0
+Text GLabel 6450 1400 2    50   Input ~ 0
 COL3
-Text GLabel 6350 3200 2    50   Input ~ 0
+Text GLabel 6450 1500 2    50   Input ~ 0
 COL4
+Text GLabel 6450 1600 2    50   Input ~ 0
+COL5
+Text GLabel 6350 2000 2    50   Input ~ 0
+COL6
+Text GLabel 6350 3700 2    50   Input ~ 0
+ENCR1
+Text GLabel 6350 3800 2    50   Input ~ 0
+ENCR2
+Text GLabel 6350 1800 2    50   Input ~ 0
+ENCL1
 Text GLabel 6350 1700 2    50   Input ~ 0
-COL5
-Text GLabel 6350 1800 2    50   Input ~ 0
-COL6
-Text GLabel 6350 3900 2    50   Input ~ 0
-ENCR1
-Text GLabel 6350 4000 2    50   Input ~ 0
-ENCR2
-Text GLabel 6350 4200 2    50   Input ~ 0
-ENCL1
-Text GLabel 6350 4100 2    50   Input ~ 0
 ENCL2
-Text GLabel 6350 1900 2    50   Input ~ 0
+Text GLabel 6350 2700 2    50   Input ~ 0
 LED
 Wire Wire Line
@@
 Wire Wire Line
 	3200 8950 3200 8900
-Text GLabel 6450 1600 2    50   Input ~ 0
+Text GLabel 6350 4000 2    50   Input ~ 0
 ROWR0
 Text GLabel 6350 1300 2    50   Input ~ 0
 ROWR3
-Text GLabel 6450 1400 2    50   Input ~ 0
+Text GLabel 6350 3500 2    50   Input ~ 0
 ROWR2
-Text GLabel 6450 1500 2    50   Input ~ 0
+Text GLabel 6350 3900 2    50   Input ~ 0
 ROWR1
-Text GLabel 6600 2700 2    50   Input ~ 0
+Text GLabel 6350 2200 2    50   Input ~ 0
 ROWL1
+Text GLabel 6350 1900 2    50   Input ~ 0
+ROWL2
+Text GLabel 6350 2800 2    50   Input ~ 0
+ROWL3
+Wire Wire Line
+	8200 7500 9000 7500
 Text GLabel 6350 2300 2    50   Input ~ 0
-ROWL2
-Text GLabel 6350 2200 2    50   Input ~ 0
-ROWL3
-Wire Wire Line
-	8200 7500 9000 7500
-Text GLabel 6600 2000 2    50   Input ~ 0
 ROWL0
 Text GLabel 6850 1650 2    50   Input ~ 0
@@
 Wire Wire Line
 	6100 7950 6500 7950
-Text GLabel 6350 3700 2    50   Input ~ 0
+Text GLabel 6350 3100 2    50   Input ~ 0
 JOYSTX
 Text GLabel 6500 8100 0    50   Input ~ 0
 JOYSTX
-Text GLabel 6350 3800 2    50   Input ~ 0
+Text GLabel 6350 2900 2    50   Input ~ 0
 JOYSTY
 Text GLabel 6500 7650 0    50   Input ~ 0
 JOYSTY
-Wire Wire Line
-	6350 2000 6600 2000
-Wire Wire Line
-	6350 2700 6600 2700
-Text GLabel 6600 3500 2    50   Input ~ 0
+Text GLabel 6350 3200 2    50   Input ~ 0
 JOYSTBT
-Wire Wire Line
-	6350 3500 6600 3500
 Text GLabel 6500 7800 0    50   Input ~ 0
 JOYSTBT

Commit message: update yacc46 schematic and footprints
Parts:
- removed J3: joystick_switch_joycon, 1m38_kbd:Molex_FPC_CON_0.5mm_5pin_5051100592, symbol 1m38_kbd:joystick_switch_joycon
- SW19, SW36: footprint 1m38_kbd:RotaryEncoder_Alps_EC11E-and-CherryMX-Single -> 1m38_kbd:RotaryEncoder_Alps_EC11E-and-CherryMX-Hotswap
- renumbered J4 to J3, J5 to J4, D47 to U2
Connections:
- net JOYSTBT: no longer names the net of U1.27 (PD7)
- net JOYSTX: no longer names the net of U1.26 (PD6)
- net JOYSTY: no longer names the net of U1.25 (PD4)
- no-connect marks 3 -> 6
Changed lines of the file:
@@
 F 0 "SW19" H 13750 3050 50  0000 L CNN
 F 1 "Rotary_Encoder_Switch" H 13150 3150 50  0000 L CNN
-F 2 "1m38_kbd:RotaryEncoder_Alps_EC11E-and-CherryMX-Single" H 13800 2960 50  0001 C CNN
+F 2 "1m38_kbd:RotaryEncoder_Alps_EC11E-and-CherryMX-Hotswap" H 13800 2960 50  0001 C CNN
 F 3 "~" H 13950 3060 50  0001 C CNN
 	1    13950 2800
@@
 F 0 "SW36" H 8750 6250 50  0000 L CNN
 F 1 "Rotary_Encoder_Switch" H 7850 6250 50  0000 L CNN
-F 2 "1m38_kbd:RotaryEncoder_Alps_EC11E-and-CherryMX-Single" H 8600 6660 50  0001 C CNN
+F 2 "1m38_kbd:RotaryEncoder_Alps_EC11E-and-CherryMX-Hotswap" H 8600 6660 50  0001 C CNN
 F 3 "~" H 8750 6760 50  0001 C CNN
 	1    8750 6500
@@
 $EndComp
 $Comp
-L Connector:AVR-ISP-6 J4
+L Connector:AVR-ISP-6 J3
 U 1 1 5F784B6C
 P 1500 9000
-F 0 "J4" H 1171 9096 50  0000 R CNN
+F 0 "J3" H 1171 9096 50  0000 R CNN
 F 1 "AVR-ISP-6" H 1171 9005 50  0000 R CNN
 F 2 "1m38_kbd:ICSP-Header-ZigZag-Single" V 1250 9050 50  0001 C CNN
@@
 	3000 8900 3000 9000
 $Comp
-L Connector_Generic:Conn_01x04 J5
+L Connector_Generic:Conn_01x04 J4
 U 1 1 5F59F101
 P 2800 8700
-F 0 "J5" V 3000 8400 50  0000 R CNN
+F 0 "J4" V 3000 8400 50  0000 R CNN
 F 1 "GLOVE_I2C" V 2900 8400 50  0000 R CNN
 F 2 "1m38_kbd:Grove_I2C" H 2800 8700 50  0001 C CNN
@@
 	1700 5800 2000 5800
 $Comp
-L Power_Protection:PRTR5V0U2X D47
+L Power_Protection:PRTR5V0U2X U2
 U 1 1 60347A24
 P 3250 3950
-F 0 "D47" V 3296 3406 50  0000 R CNN
+F 0 "U2" V 3296 3406 50  0000 R CNN
 F 1 "PRTR5V0U2X" V 3205 3406 50  0000 R CNN
 F 2 "1m38_kbd:PRTR5V0U2X_SOT143B" H 3310 3950 50  0001 C CNN
@@
 Wire Wire Line
 	4550 9500 4550 10050
-$Comp
-L 1m38_kbd:joystick_switch_joycon J3
-U 1 1 609C0DD2
-P 7050 7800
-F 0 "J3" H 7478 7846 50  0000 L CNN
-F 1 "joystick_switch_joycon" H 7478 7755 50  0000 L CNN
-F 2 "1m38_kbd:Molex_FPC_CON_0.5mm_5pin_5051100592" H 6850 7750 50  0001 C CNN
-F 3 "" H 6850 7750 50  0001 C CNN
-	1    7050 7800
-	1    0    0    -1
-$EndComp
-$Comp
-L power:GND #PWR0107
-U 1 1 609C2EA8
-P 6100 7950
-F 0 "#PWR0107" H 6100 7700 50  0001 C CNN
-F 1 "GND" H 6105 7777 50  0000 C CNN
-F 2 "" H 6100 7950 50  0001 C CNN
-F 3 "" H 6100 7950 50  0001 C CNN
-	1    6100 7950
-	1    0    0    -1
-$EndComp
-$Comp
-L power:VCC #PWR0108
-U 1 1 609C381E
-P 6100 7500
-F 0 "#PWR0108" H 6100 7350 50  0001 C CNN
-F 1 "VCC" H 6115 7673 50  0000 C CNN
-F 2 "" H 6100 7500 50  0001 C CNN
-F 3 "" H 6100 7500 50  0001 C CNN
-	1    6100 7500
-	1    0    0    -1
-$EndComp
-Wire Wire Line
-	6100 7500 6500 7500
-Wire Wire Line
-	6100 7950 6500 7950
-Text GLabel 6350 3100 2    50   Input ~ 0
-JOYSTX
-Text GLabel 6500 8100 0    50   Input ~ 0
-JOYSTX
-Text GLabel 6350 2900 2    50   Input ~ 0
-JOYSTY
-Text GLabel 6500 7650 0    50   Input ~ 0
-JOYSTY
-Text GLabel 6350 3200 2    50   Input ~ 0
-JOYSTBT
-Text GLabel 6500 7800 0    50   Input ~ 0
-JOYSTBT
+NoConn ~ 6350 2900
+NoConn ~ 6350 3100
+NoConn ~ 6350 3200
 $EndSCHEMATC
