File: yacc46/yacc46.kicad_pcb (KiCad board)
At the start: 2 copper layers, 285.5 x 112.1 mm, 144 parts, among them J1 USB_C_Receptacle_USB2.0, J2 OLED_I2C, J3 joystick_switch_joycon, J4 AVR-ISP-6, J5 GLOVE_I2C, SW1 SW_PUSH, SW10 SW_PUSH, SW11 SW_PUSH, SW12 SW_PUSH, SW13 SW_PUSH, SW14 SW_PUSH, SW15 SW_PUSH, SW16 SW_PUSH, SW17 SW_PUSH, SW18 SW_PUSH, SW19 Rotary_Encoder_Switch, SW2 SW_PUSH, SW20 SW_PUSH, SW21 SW_PUSH, SW22 SW_PUSH, SW23 SW_PUSH, SW24 SW_PUSH, SW25 SW_PUSH, SW26 SW_PUSH, SW27 SW_PUSH, SW28 SW_PUSH, SW29 SW_PUSH, SW3 SW_PUSH, SW30 SW_PUSH, SW31 SW_PUSH, SW32 SW_PUSH, SW33 SW_PUSH, SW34 SW_PUSH, SW35 SW_PUSH, SW36 Rotary_Encoder_Switch, SW37 SW_PUSH, SW38 SW_PUSH, SW39 SW_PUSH, SW4 SW_PUSH, SW40 SW_PUSH, SW41 SW_PUSH, SW42 SW_PUSH, SW43 SW_PUSH, SW44 SW_PUSH, SW45 SW_PUSH, SW46 SW_PUSH, SW47 SW_Push, SW5 SW_PUSH, SW6 SW_PUSH, SW7 SW_PUSH, SW8 SW_PUSH, SW9 SW_PUSH, U1 ATmega32U4-AU, Y1 16MHz

Commit message: [WIP]配線中
Parts:
- moved F1 178.1 mm to (116.5, 32.9)
- moved R1 170.7 mm to (157.4, 31.5), turned to 90 degrees
- moved J4 168.0 mm to (211.1, 27.7), turned to 270 degrees
- moved D47 165.4 mm to (134.0, 39.9)
- moved R2 158.2 mm to (160.1, 31.5), turned to 270 degrees
- moved J5 132.1 mm to (206.6, 34.4), turned to 270 degrees
- moved C2 118.8 mm to (165.9, 81.1), turned to 270 degrees
- moved C4 118.7 mm to (170.6, 81.1), turned to 90 degrees
- moved R4 115.6 mm to (175.8, 81.1), turned to 90 degrees
- moved C3 114.6 mm to (168.3, 81.1), turned to 90 degrees
- moved R3 113.9 mm to (173.5, 81.1), turned to 90 degrees
- moved C1 110.8 mm to (163.5, 81.1), turned to 270 degrees
- moved C6 89.3 mm to (171.3, 112.8), turned to 90 degrees
- moved C5 84.8 mm to (161.2, 112.8), turned to 270 degrees
- moved Y1 80.0 mm to (166.3, 112.8), turned to 180 degrees
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Routing:
- net GND: track 0.00 -> 786.1 mm, vias 0 -> 12
- net VBUS: track 0.00 -> 777.1 mm
- net COL3: track 0.00 -> 231.2 mm, vias 0 -> 3
- net ROWL1: track 0.00 -> 142.2 mm, vias 0 -> 3
- net MOSI: track 0.00 -> 141.2 mm, vias 0 -> 1
- net ROWL2: track 0.00 -> 139.0 mm, vias 0 -> 3
- net ROWR2: track 0.00 -> 138.5 mm, vias 0 -> 3
- net COL4: track 0.00 -> 129.6 mm, vias 0 -> 1
- net COL5: track 0.00 -> 126.2 mm, vias 0 -> 1
- net MISO: track 0.00 -> 107.1 mm, vias 0 -> 7
- net ROWL0: track 0.00 -> 105.9 mm, vias 0 -> 5
- net UDN: track 0.00 -> 99.8 mm, vias 0 -> 4
- net UDP: track 0.00 -> 99.1 mm, vias 0 -> 3
- net COL6: track 0.00 -> 96.6 mm, vias 0 -> 1
- net Net-(LED6-Pad2): track 0.00 -> 83.8 mm, vias 0 -> 2
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Other:
- outline, holes or cut-outs redrawn
- board text added: "RESET"
