File: yacc46/yacc46_plate.kicad_pcb (KiCad board)
At the start: 2 copper layers, 281.1 x 112.1 mm, 141 parts, among them J1 CX70M-24P1, J2 OLED_I2C, J3 AVR-ISP-6, J4 GLOVE_I2C, J5 TRRS_I2C, SW1 SW_PUSH, SW10 SW_PUSH, SW11 SW_PUSH, SW12 SW_PUSH, SW13 SW_PUSH, SW14 SW_PUSH, SW15 SW_PUSH, SW16 SW_PUSH, SW17 SW_PUSH, SW18 SW_PUSH, SW19 Rotary_Encoder_Switch, SW2 SW_PUSH, SW20 SW_PUSH, SW21 SW_PUSH, SW22 SW_PUSH, SW23 SW_PUSH, SW24 SW_PUSH, SW25 SW_PUSH, SW26 SW_PUSH, SW27 SW_PUSH, SW28 SW_PUSH, SW29 SW_PUSH, SW3 SW_PUSH, SW30 SW_PUSH, SW31 SW_PUSH, SW32 SW_PUSH, SW33 SW_PUSH, SW34 SW_PUSH, SW35 SW_PUSH, SW36 Rotary_Encoder_Switch, SW37 SW_PUSH, SW38 SW_PUSH, SW39 SW_PUSH, SW4 SW_PUSH, SW40 SW_PUSH, SW41 SW_PUSH, SW42 SW_PUSH, SW43 SW_PUSH, SW44 SW_PUSH, SW45 SW_PUSH, SW46 SW_PUSH, SW5 SW_PUSH, SW6 SW_PUSH, SW7 SW_PUSH, SW8 SW_PUSH, SW9 SW_PUSH, U1 ATmega32U4-AU, Y1 16MHz

Commit message: プレート元データを作成
Parts:
- removed the HOLE13 at (152.0, 60.1)
- removed the HOLE13 at (164.8, 88.2)
- removed J5: TRRS_I2C, 1m38_kbd:MJ-4PP-9_1side_no-mask
- added HOLE13: Val**, 1m38_kbd:M2_ScrewHole, F.Cu at (165.0, 80.1)
- added HOLE15: M2_ScrewHole, 1m38_kbd:M2_ScrewHole, F.Cu at (178.0, 60.1)
- added SW47: SW_Push, 1m38_kbd:SW_PUSH_SMD_TVAF06-A020B-R_HandSolder, B.Cu at (184.1, 132.6)
- C1, C2, C3, C4: footprint Capacitor_SMD:C_0805_2012Metric_Pad1.15x1.40mm_HandSolder -> Capacitor_SMD:C_0805_2012Metric_Pad1.18x1.45mm_HandSolder
- C5, C6: footprint Capacitor_SMD:C_0603_1608Metric_Pad1.05x0.95mm_HandSolder -> Capacitor_SMD:C_0603_1608Metric_Pad1.08x0.95mm_HandSolder
- HOLE1, HOLE10, HOLE11, HOLE12, HOLE2, HOLE3, HOLE4, HOLE5, HOLE6, HOLE7, HOLE8, HOLE9: footprint foostan-kbd:M2_HOLE_v2 -> 1m38_kbd:M2_ScrewHole
- HOLE14: value MountingHole_2.2mm_M2 -> M2_ScrewHole; footprint MountingHole:MountingHole_2.2mm_M2 -> 1m38_kbd:M2_ScrewHole
- R1, R2, R3, R4, R5, R6: footprint Resistor_SMD:R_0805_2012Metric_Pad1.15x1.40mm_HandSolder -> Resistor_SMD:R_0805_2012Metric_Pad1.20x1.40mm_HandSolder
- Y1: footprint Crystal:Crystal_SMD_2520-4Pin_2.5x2.0mm -> Crystal:Crystal_SMD_SeikoEpson_FA238-4Pin_3.2x2.5mm_HandSoldering
- moved J4 78.5 mm to (205.6, 34.1), turned to 270 degrees
- moved HOLE14 25.5 mm to (152.0, 60.1)
- moved C1 13.8 mm to (161.0, 96.7)
- moved C2 13.7 mm to (163.3, 96.7)
- moved C3 13.6 mm to (165.7, 96.7)
- moved C4 13.6 mm to (168.1, 96.7)
- moved R3 12.3 mm to (165.6, 90.1)
- moved R4 12.3 mm to (168.1, 90.1)
- moved U1 11.1 mm to (165.0, 111.2)
- moved C5 10.7 mm to (167.3, 125.7), turned to 270 degrees
- moved Y1 10.2 mm to (172.0, 125.7)
- moved R5 8.86 mm to (177.5, 132.6)
- moved C6 8.65 mm to (176.6, 125.7), turned to 90 degrees
- moved D35 5.33 mm to (302.4, 71.9)
- moved D42 5.33 mm to (302.4, 90.9)
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Connections:
- Y1 pad 1: XTAL1 -> XTAL2
- Y1 pad 3: XTAL2 -> XTAL1
Other:
- board size 281.1 x 112.1 mm -> 281.5 x 112.1 mm
- rule pad_to_mask_clearance: 0.05 -> 0
- board text added: "RESET"
- board text added: "yacc46 v0.2 PCB designed by 1.038"
- board text removed: "yacc46 v0.1 PCB designed by 1.038"

Commit message: ロータリーエンコーダ兼用スイッチ穴のフットプリントを修正
Parts:
- SW19, SW36: footprint 1m38_kbd:CherryMX_SwitchHole_RoundCorner -> 1m38_kbd:EC11E-and-CherryMX_SwitchHole_RoundCorner

Commit message: sandwitchプレートデータを作成
Parts:
- removed HOLE1, HOLE10, HOLE11, HOLE12, HOLE13, HOLE2, HOLE3, HOLE4, HOLE5, HOLE6, HOLE7, HOLE8, HOLE9: Val**, 1m38_kbd:M2_ScrewHole
- removed HOLE14, HOLE15: M2_ScrewHole, 1m38_kbd:M2_ScrewHole
- added D47: PRTR5V0U2X, 1m38_kbd:PRTR5V0U2X_SOT143B, B.Cu at (134.0, 39.9)
- added H1: MountingHole, 1m38_kbd:M2_ScrewHole, F.Cu at (132.0, 132.9)
- added H10: MountingHole, 1m38_kbd:M2_ScrewHole, F.Cu at (292.0, 95.8)
- added H11: MountingHole, 1m38_kbd:M2_ScrewHole, F.Cu at (249.6, 102.5)
- added H12: MountingHole, 1m38_kbd:M2_ScrewHole, F.Cu at (202.0, 132.9)
- added H13: MountingHole, 1m38_kbd:M2_ScrewHole, F.Cu at (153.4, 60.1)
- added H14: MountingHole, 1m38_kbd:M2_ScrewHole, F.Cu at (180.6, 60.1)
- added H2: MountingHole, 1m38_kbd:M2_ScrewHole, F.Cu at (84.4, 102.5)
- added H3: MountingHole, 1m38_kbd:M2_ScrewHole, F.Cu at (42.0, 95.8)
- added H4: MountingHole, 1m38_kbd:M2_ScrewHole, F.Cu at (34.7, 46.2)
- added H5: MountingHole, 1m38_kbd:M2_ScrewHole, F.Cu at (86.2, 30.9)
- added H6: MountingHole, 1m38_kbd:M2_ScrewHole, F.Cu at (142.0, 30.9)
- added H7: MountingHole, 1m38_kbd:M2_ScrewHole, F.Cu at (192.0, 30.9)
- added H8: MountingHole, 1m38_kbd:M2_ScrewHole, F.Cu at (247.8, 30.9)
- added H9: MountingHole, 1m38_kbd:M2_ScrewHole, F.Cu at (299.3, 46.2)
- added HOLE_ST: Switch_Joycon_Joystick_FPC_hole, 1m38_kbd:Switch_Joycon_Joystick_FPC_hole, F.Cu at (154.3, 132.2)
- added J5: GLOVE_I2C, 1m38_kbd:Grove_I2C, F.Cu at (206.6, 34.4)
- added ST1: Switch_Joycon_Joystick, 1m38_kbd:Switch_Joycon_Joystick, F.Cu at (167.0, 120.5)
- J1: value CX70M-24P1 -> USB_C_Receptacle_USB2.0; footprint digikey-footprints:USB-C_Female_CX70M-24P1 -> 1m38_kbd:USB-C_Female_CX90M-16P
- J3: value AVR-ISP-6 -> joystick_switch_joycon; footprint 1m38_kbd:ICSP-Header-ZigZag-Single -> 1m38_kbd:Molex_FPC_CON_0.5mm_5pin_5051100592
- J4: value GLOVE_I2C -> AVR-ISP-6; footprint 1m38_kbd:Grove_I2C -> 1m38_kbd:ICSP-Header-ZigZag-Single; moved to B.Cu
- LED1, LED10, LED11, LED12, LED13, LED14, LED2, LED3, LED4, LED5, LED6, LED7, LED8, LED9: value WS2813 -> WS2812B; footprint LED_SMD:LED_WS2812_PLCC6_5.0x5.0mm_P1.6mm -> foostan_kbd:LED_WS2812B-PLCC4
- moved R1 115.5 mm to (153.7, 29.4), turned to 0 degrees
- moved R2 115.5 mm to (153.7, 31.7), turned to 180 degrees
- moved J3 103.0 mm to (154.3, 124.3), turned to 180 degrees
- moved J1 99.0 mm to (128.4, 32.4), turned to 180 degrees
- moved F1 66.5 mm to (116.5, 32.9), turned to 0 degrees
- moved R6 17.5 mm to (169.6, 133.2), turned to 180 degrees
- moved D19 17.3 mm to (138.5, 95.3)
- moved C5 15.9 mm to (161.3, 111.0)
- moved Y1 15.8 mm to (166.4, 111.0)
- moved C4 15.7 mm to (170.6, 81.1)
- moved C3 15.7 mm to (168.3, 81.1)
- moved C2 15.7 mm to (165.9, 81.1)
- moved C1 15.7 mm to (163.5, 81.1)
- moved C6 15.6 mm to (171.5, 111.0)
- moved R3 15.3 mm to (168.4, 75.0)
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Connections:
- D24 pad 1: MISO -> ROWR0
- D25 pad 1: MISO -> ROWR0
- D26 pad 1: MISO -> ROWR0
- D27 pad 1: MISO -> ROWR0
- D28 pad 1: MISO -> ROWR0
- D29 pad 1: MOSI -> ROWR1
- D30 pad 1: MOSI -> ROWR1
- D31 pad 1: MOSI -> ROWR1
- D32 pad 1: MOSI -> ROWR1
- D33 pad 1: MOSI -> ROWR1
- D34 pad 1: MOSI -> ROWR1
- D35 pad 1: MOSI -> ROWR1
- J1 pad A5: /CC1 -> Net-(J1-PadA5)
- J1 pad A8: Net-(J1-PadA8) -> (no net)
- J1 pad B5: /CC2 -> Net-(J1-PadB5)
- J1 pad B8: Net-(J1-PadB8) -> (no net)
- J3 pad 1: MISO -> JOYSTX
- J3 pad 2: VBUS -> GND
- J3 pad 3: ROWR2 -> JOYSTBT
- J3 pad 4: MOSI -> JOYSTY
- J3 pad 5: RESET -> VBUS
- J4 pad 1: SDA -> COL5
- J4 pad 2: SCL -> VBUS
- J4 pad 3: VBUS -> COL3
- J4 pad 4: GND -> COL4
- LED1 pad 1: Net-(LED1-Pad1) -> VBUS
- LED1 pad 2: VBUS -> Net-(LED1-Pad2)
- LED1 pad 3: Net-(LED1-Pad3) -> GND
- LED10 pad 1: Net-(LED10-Pad1) -> VBUS
- LED10 pad 2: VBUS -> Net-(LED10-Pad2)
- LED10 pad 3: Net-(LED10-Pad3) -> GND
- LED11 pad 1: Net-(LED11-Pad1) -> VBUS
- LED11 pad 2: VBUS -> Net-(LED11-Pad2)
- LED11 pad 3: Net-(LED11-Pad3) -> GND
- LED11 pad 4: Net-(LED10-Pad3) -> Net-(LED10-Pad2)
- LED12 pad 1: Net-(LED12-Pad1) -> VBUS
- LED12 pad 2: VBUS -> Net-(LED12-Pad2)
- LED12 pad 3: Net-(LED12-Pad3) -> GND
- LED12 pad 4: Net-(LED11-Pad3) -> Net-(LED11-Pad2)
- LED13 pad 1: Net-(LED13-Pad1) -> VBUS
- LED13 pad 2: VBUS -> Net-(LED13-Pad2)
- LED13 pad 3: Net-(LED13-Pad3) -> GND
- LED13 pad 4: Net-(LED12-Pad3) -> Net-(LED12-Pad2)
- LED14 pad 1: Net-(LED14-Pad1) -> VBUS
- LED14 pad 2: VBUS -> (no net)
- LED14 pad 3: Net-(LED14-Pad3) -> GND
- LED14 pad 4: Net-(LED13-Pad3) -> Net-(LED13-Pad2)
- LED2 pad 1: Net-(LED2-Pad1) -> VBUS
- LED2 pad 2: VBUS -> Net-(LED2-Pad2)
- LED2 pad 3: Net-(LED2-Pad3) -> GND
- LED2 pad 4: Net-(LED1-Pad3) -> Net-(LED1-Pad2)
- LED3 pad 1: Net-(LED3-Pad1) -> VBUS
- LED3 pad 2: VBUS -> Net-(LED3-Pad2)
- LED3 pad 3: Net-(LED3-Pad3) -> GND
- LED3 pad 4: Net-(LED2-Pad3) -> Net-(LED2-Pad2)
- LED4 pad 1: Net-(LED4-Pad1) -> VBUS
- LED4 pad 2: VBUS -> Net-(LED4-Pad2)
- LED4 pad 3: Net-(LED4-Pad3) -> GND
- LED4 pad 4: Net-(LED3-Pad3) -> Net-(LED3-Pad2)
- LED5 pad 1: Net-(LED5-Pad1) -> VBUS
- LED5 pad 2: VBUS -> Net-(LED5-Pad2)
- LED5 pad 3: Net-(LED5-Pad3) -> GND
- LED5 pad 4: Net-(LED4-Pad3) -> Net-(LED4-Pad2)
- LED6 pad 1: Net-(LED6-Pad1) -> VBUS
- LED6 pad 2: VBUS -> Net-(LED6-Pad2)
- LED6 pad 3: Net-(LED6-Pad3) -> GND
- LED6 pad 4: Net-(LED5-Pad3) -> Net-(LED5-Pad2)
- LED7 pad 1: Net-(LED7-Pad1) -> VBUS
- LED7 pad 2: VBUS -> Net-(LED7-Pad2)
- LED7 pad 3: Net-(LED7-Pad3) -> GND
- LED7 pad 4: Net-(LED6-Pad3) -> Net-(LED6-Pad2)
- LED8 pad 1: Net-(LED8-Pad1) -> VBUS
- LED8 pad 2: VBUS -> Net-(LED8-Pad2)
- LED8 pad 3: Net-(LED10-Pad6) -> GND
- LED8 pad 4: Net-(LED7-Pad3) -> Net-(LED7-Pad2)
- LED9 pad 1: Net-(LED9-Pad1) -> VBUS
- LED9 pad 2: VBUS -> Net-(LED10-Pad4)
- LED9 pad 3: Net-(LED10-Pad4) -> GND
- LED9 pad 4: Net-(LED10-Pad6) -> Net-(LED8-Pad2)
- R1 pad 1: GND -> Net-(J1-PadA5)
- R1 pad 2: /CC1 -> GND
- R2 pad 1: /CC2 -> GND
- R2 pad 2: GND -> Net-(J1-PadB5)
- R4 pad 1: UDP -> DP
- R4 pad 2: DP -> UDP
- U1 pad 1: Net-(U1-Pad1) -> ROWR2
- U1 pad 10: MOSI -> COL4
- U1 pad 11: MISO -> COL5
- U1 pad 12: Net-(U1-Pad12) -> COL6
- U1 pad 20: Net-(U1-Pad20) -> LED
- U1 pad 21: COL0 -> ROWL3
- U1 pad 22: COL1 -> COL0
- U1 pad 25: COL2 -> JOYSTY
- U1 pad 26: COL3 -> JOYSTX
- U1 pad 27: COL4 -> JOYSTBT
- U1 pad 28: COL5 -> ENCL2
- U1 pad 29: COL6 -> ENCL1
- U1 pad 30: LED -> ROWL2
- U1 pad 31: ROWL3 -> ROWL1
- U1 pad 32: ROWL2 -> ROWL0
- U1 pad 36: ROWL1 -> COL1
- U1 pad 37: ROWL0 -> COL2
- U1 pad 38: ENCL1 -> ROWR0
- U1 pad 39: ENCL2 -> ROWR1
- U1 pad 9: ROWR2 -> COL3
Routing:
- net VBUS: track 0.00 -> 764.7 mm
- net GND: track 0.00 -> 670.4 mm, vias 0 -> 187
- net COL0: track 0.00 -> 392.1 mm, vias 0 -> 7
- net COL3: track 0.00 -> 389.9 mm, vias 0 -> 13
- net COL1: track 0.00 -> 362.2 mm, vias 0 -> 8
- net COL4: track 0.00 -> 324.5 mm, vias 0 -> 8
- net COL2: track 0.00 -> 305.4 mm, vias 0 -> 6
- net COL5: track 0.00 -> 303.5 mm, vias 0 -> 9
- net RESET: track 0.00 -> 191.8 mm, vias 0 -> 6
- net ROWR2: track 0.00 -> 173.4 mm, vias 0 -> 4
- net COL6: track 0.00 -> 172.9 mm, vias 0 -> 5
- net ROWR1: track 0.00 -> 172.4 mm, vias 0 -> 2
- net ROWR0: track 0.00 -> 171.0 mm, vias 0 -> 8
- net ROWL2: track 0.00 -> 162.4 mm, vias 0 -> 4
- net ROWL0: track 0.00 -> 157.0 mm, vias 0 -> 6
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- added copper zone on B.Cu, net GND
- added copper zone on F.Cu, net GND
Other:
- board size 281.5 x 112.1 mm -> 285.5 x 112.1 mm
- net class Default: clearance 0.2 -> 0.2032
- net class Power: clearance 0.2 -> 0.2032
- rule trace_clearance: 0.2 -> 0.2032
- board text added: "yacc46 v0.3 PCB designed by 1.038"
- board text removed: "yacc46 v0.2 PCB designed by 1.038"
