File: yacc46/plate_v0.4/top_pcb/yacc46_plate.kicad_pcb (KiCad board)
At the start: 2 copper layers, 291.6 x 112.1 mm, 59 parts, among them SW1 SW_PUSH, SW10 SW_PUSH, SW11 SW_PUSH, SW12 SW_PUSH, SW13 SW_PUSH, SW14 SW_PUSH, SW15 SW_PUSH, SW16 SW_PUSH, SW17 SW_PUSH, SW18 SW_PUSH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

Commit message: yacc46 v1.0 plate: add copper on the back side
Routing:
- added copper zone on B.Cu, net (none)
